File: Senior_Design_Lab1_Team3.kicad_sch (KiCad schematic)
At the start: 18 parts, among them J1 Raspberry_Pi_4, SW1 SPDT Toggle Switch, U1 Temperature Sensor 1, U2 Temperature Sensor 2, U3 LCD1602

Commit message: Add files via upload
Parts:
- added R10, R11: 4.7KΩ, symbol Device:R_Small_US
Connections:
- net +5V: now also R10.1, R11.1
- net at J1.11 (GPIO17), U2.1 (Data): now also R10.2
- net at J1.7 (GPIO4), U1.1 (Data): now also R11.2
